Commit message: First draft for Humble

File: hyperdog_gazebo_sim/description/gazebo_ros2_control_plugin.xacro (robot description, xacro)
@@ -1,11 +1,4 @@
 <?xml version="1.0"?>
 <robot xmlns:xacro="http://www.ros.org/wiki/xacro">
-<!-- ************* JOINT CONTROLLER GAZEBO PLUGIN ************** -->
-    <!--
-    _____________________________________________________________________
-        include this file into: /description/hyperdog.urdf.xacro
-        using following line:
-                    <xacro:include filename="gazebo_ros2_control_plugin.xacro" />
-    _____________________________________________________________________ -->
     <!-- CONFIGURE JOINTS OF THE ROBOT -->
     <ros2_control name="GazeboSystem" type="System">
@@ -36,4 +29,8 @@
         </joint>
         <joint name="FR_lleg_joint">
+            <param name="pos_kp">100000</param>
+            <param name="pos_ki">0</param>
+            <param name="pos_kd">0</param>
+            <param name="pos_max_integral_error">10000</param>
             <command_interface name="position">
                 <param name="min">0.45</param>
@@ -69,4 +66,8 @@
         </joint>
         <joint name="FL_lleg_joint">
+            <param name="pos_kp">200000</param>
+            <param name="pos_ki">0</param>
+            <param name="pos_kd">0</param>
+            <param name="pos_max_integral_error">10000</param>
             <command_interface name="position">
                 <param name="min">0.45</param>
@@ -102,4 +103,8 @@
         </joint>
         <joint name="BR_lleg_joint">
+            <param name="pos_kp">300000</param>
+            <param name="pos_ki">0</param>
+            <param name="pos_kd">0</param>
+            <param name="pos_max_integral_error">10000</param>
             <command_interface name="position">
                 <param name="min">0.45</param>
@@ -135,4 +140,8 @@
         </joint>
         <joint name="BL_lleg_joint">
+            <param name="pos_kp">500000</param>
+            <param name="pos_ki">0</param>
+            <param name="pos_kd">0</param>
+            <param name="pos_max_integral_error">10000</param>
             <command_interface name="position">
                 <param name="min">0.45</param>

File: hyperdog_gazebo_sim/description/hyperdog_gazebo.xacro (robot description, xacro)
@@ -1,13 +1,4 @@
 <?xml version="1.0"?>
 <robot xmlns:xacro="http://www.ros.org/wiki/xacro">
-<!--
-    _____________________________________________________________________
-        include this file into: /description/hyperdog.urdf.xacro
-        using following line:
-                    <xacro:include filename="hyperdog_gazebo.xacro" />
-    _____________________________________________________________________
-    * Gazebo is unable to use the same <material> tags that are already in the URDF (that RViz uses).
-    Instead, we need to add gazebo tags for our links that refer to Gazebo materials
--->
     <xacro:include filename="physics.xacro" />
     <xacro:macro name="gz_hip">
@@ -47,8 +38,10 @@
         <mu1>0.9</mu1>
         <mu2>0.9</mu2>
-        <fdir1>1 1 0</fdir1>
+        <fdir1>1 0 0</fdir1>
         <kp value="2147483647.0" />
         <kd value="100.0" />
-        <maxVel>0.01</maxVel>
+        <maxVel>0.0</maxVel>
+        <maxContacts>1</maxContacts>
+        <gravity>true</gravity>
         <self_collide>1</self_collide>
         <minDepth>0.001</minDepth>

File: hyperdog_gazebo_sim/description/hyperdog_urdf_joints.xacro (robot description, xacro)
@@ -1,10 +1,4 @@
 <?xml version="1.0"?>
 <robot xmlns:xacro="http://www.ros.org/wiki/xacro">
-<!--
-    _____________________________________________________________________
-        include this file into: /description/hyperdog.urdf.xacro
-        using following line:
-                    <xacro:include filename="hyperdog_urdf_joints.xacro" />
-    _____________________________________________________________________ -->
     <xacro:include filename="consts.xacro" />
     <!-- Limits -->

File: hyperdog_gazebo_sim/description/hyperdog_urdf_links.xacro (robot description, xacro)
@@ -1,12 +1,4 @@
 <?xml version="1.0"?>
 <robot xmlns:xacro="http://www.ros.org/wiki/xacro">
-<!--
-    * Autor: nipun.dhananjaya@gmail.com
-    * Date:  13.03.2023
-    _____________________________________________________________________
-        include this file into: /description/hyperdog.urdf.xacro
-        using following line:
-                    <xacro:include filename="hyperdog_urdf_links.xacro" />
-    _____________________________________________________________________ -->
     <xacro:include filename="consts.xacro" />
     <xacro:include filename="physics.xacro" />
